Commit message: fix: Update the URDF and SRDF files to include the new self-collision links for the fr3_duo robot

File: franka_selfcollision/test/fr3_duo.urdf (robot description, URDF)
Before this commit: robot fr3_duo, 46 links, 45 joints
Links:
- removed link left_fr3_link0
- removed link left_fr3_link0_accelerometer_bottom
- removed link left_fr3_link0_accelerometer_top
- removed link left_fr3_link1
- removed link left_fr3_link1_accelerometer_bottom
- removed link left_fr3_link1_accelerometer_top
- removed link left_fr3_link2
- removed link left_fr3_link2_accelerometer_bottom
- removed link left_fr3_link2_accelerometer_top
- removed link left_fr3_link3
- removed link left_fr3_link3_accelerometer_bottom
- removed link left_fr3_link3_accelerometer_top
- removed link left_fr3_link4
- removed link left_fr3_link4_accelerometer_bottom
- removed link left_fr3_link4_accelerometer_top
- removed link left_fr3_link5
- removed link left_fr3_link5_accelerometer_bottom
- removed link left_fr3_link5_accelerometer_top
- removed link left_fr3_link6
- removed link left_fr3_link7
- removed link left_fr3_link8
- removed link mount_link
- removed link right_fr3_link0
- removed link right_fr3_link0_accelerometer_bottom
- removed link right_fr3_link0_accelerometer_top
- removed link right_fr3_link1
- removed link right_fr3_link1_accelerometer_bottom
- removed link right_fr3_link1_accelerometer_top
- removed link right_fr3_link2
- removed link right_fr3_link2_accelerometer_bottom
- removed link right_fr3_link2_accelerometer_top
- removed link right_fr3_link3
- removed link right_fr3_link3_accelerometer_bottom
- removed link right_fr3_link3_accelerometer_top
- removed link right_fr3_link4
- removed link right_fr3_link4_accelerometer_bottom
- removed link right_fr3_link4_accelerometer_top
- removed link right_fr3_link5
- removed link right_fr3_link5_accelerometer_bottom
- removed link right_fr3_link5_accelerometer_top
- removed link right_fr3_link6
- removed link right_fr3_link7
- removed link right_fr3_link8
- added link fr3_duo_mount_left
- added link fr3_duo_mount_mounting_point, mass 4.093846; collision mesh filename=package://franka_description/meshes/accessories/fr3_duo_mou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; collision mesh filename=package://franka_description/meshes/accessories/fr3_duo_mou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
- added link fr3_duo_mount_origin
- added link fr3_duo_mount_right
- added link left_fr3v2_link0, mass 2.3966; collision mesh filename=package://franka_description/meshes/robots/fr3v2/collision/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; visual mesh filename=package://franka_description/meshes/robots/fr3v2/visual/lin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
- added link left_fr3v2_link0_accelerometer_bottom
- added link left_fr3v2_link0_accelerometer_top
- added link left_fr3v2_link1, mass 2.4377; collision mesh filename=package://franka_description/meshes/robots/fr3v2/collision/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; visual mesh filename=package://franka_description/meshes/robots/fr3v2/visual/lin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
- added link left_fr3v2_link1_accelerometer_bottom
- added link left_fr3v2_link1_accelerometer_top
- added link left_fr3v2_link2, mass 2.2375; collision mesh filename=package://franka_description/meshes/robots/fr3v2/collision/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; visual mesh filename=package://franka_description/meshes/robots/fr3v2/visual/lin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
- added link left_fr3v2_link2_accelerometer_bottom
- added link left_fr3v2_link2_accelerometer_top
- added link left_fr3v2_link3, mass 2.193082; collision mesh filename=package://franka_description/meshes/robots/fr3v2/collision/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; visual mesh filename=package://franka_description/meshes/robots/fr3v2/visual/lin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
- added link left_fr3v2_link3_accelerometer_bottom
- added link left_fr3v2_link3_accelerometer_top
- added link left_fr3v2_link4, mass 2.181537; collision mesh filename=package://franka_description/meshes/robots/fr3v2/collision/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; visual mesh filename=package://franka_description/meshes/robots/fr3v2/visual/lin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
- added link left_fr3v2_link4_accelerometer_bottom
- added link left_fr3v2_link4_accelerometer_top
- added link left_fr3v2_link5, mass 2.186881; collision mesh filename=package://franka_description/meshes/robots/fr3v2/collision/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; visual mesh filename=package://franka_description/meshes/robots/fr3v2/visual/lin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
- added link left_fr3v2_link5_accelerometer_bottom
- added link left_fr3v2_link5_accelerometer_top
- added link left_fr3v2_link6, mass 1.579681; collision mesh filename=package://franka_description/meshes/robots/fr3v2/collision/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; visual mesh filename=package://franka_description/meshes/robots/fr3v2/visual/lin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
- added link left_fr3v2_link7, mass 0.694841; collision mesh filename=package://franka_description/meshes/robots/fr3v2/collision/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; visual mesh filename=package://franka_description/meshes/robots/fr3v2/visual/lin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
- added link left_fr3v2_link8
- added link right_fr3v2_link0, mass 2.3966; collision mesh filename=package://franka_description/meshes/robots/fr3v2/collision/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; visual mesh filename=package://franka_description/meshes/robots/fr3v2/visual/lin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
- added link right_fr3v2_link0_accelerometer_bottom
- added link right_fr3v2_link0_accelerometer_top
- added link right_fr3v2_link1, mass 2.4377; collision mesh filename=package://franka_description/meshes/robots/fr3v2/collision/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; visual mesh filename=package://franka_description/meshes/robots/fr3v2/visual/lin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
- added link right_fr3v2_link1_accelerometer_bottom
- added link right_fr3v2_link1_accelerometer_top
- added link right_fr3v2_link2, mass 2.2375; collision mesh filename=package://franka_description/meshes/robots/fr3v2/collision/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; visual mesh filename=package://franka_description/meshes/robots/fr3v2/visual/lin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
- added link right_fr3v2_link2_accelerometer_bottom
- added link right_fr3v2_link2_accelerometer_top
- added link right_fr3v2_link3, mass 2.193082; collision mesh filename=package://franka_description/meshes/robots/fr3v2/collision/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; visual mesh filename=package://franka_description/meshes/robots/fr3v2/visual/lin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
- added link right_fr3v2_link3_accelerometer_bottom
- added link right_fr3v2_link3_accelerometer_top
- added link right_fr3v2_link4, mass 2.181537; collision mesh filename=package://franka_description/meshes/robots/fr3v2/collision/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; visual mesh filename=package://franka_description/meshes/robots/fr3v2/visual/lin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
- added link right_fr3v2_link4_accelerometer_bottom
- added link right_fr3v2_link4_accelerometer_top
- added link right_fr3v2_link5, mass 2.186881; collision mesh filename=package://franka_description/meshes/robots/fr3v2/collision/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; visual mesh filename=package://franka_description/meshes/robots/fr3v2/visual/lin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
- added link right_fr3v2_link5_accelerometer_bottom
- added link right_fr3v2_link5_accelerometer_top
- added link right_fr3v2_link6, mass 1.579681; collision mesh filename=package://franka_description/meshes/robots/fr3v2/collision/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; visual mesh filename=package://franka_description/meshes/robots/fr3v2/visual/lin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
- added link right_fr3v2_link7, mass 0.694841; collision mesh filename=package://franka_description/meshes/robots/fr3v2/collision/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; visual mesh filename=package://franka_description/meshes/robots/fr3v2/visual/lin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
- added link right_fr3v2_link8
Joints:
- removed joint left_fr3_joint1
- removed joint left_fr3_joint2
- removed joint left_fr3_joint3
- removed joint left_fr3_joint4
- removed joint left_fr3_joint5
- removed joint left_fr3_joint6
- removed joint left_fr3_joint7
- removed joint left_fr3_joint8
- removed joint left_fr3_left_base_joint
- removed joint left_fr3_link0_accelerometer_bottom_joint
- removed joint left_fr3_link0_accelerometer_top_joint
- removed joint left_fr3_link1_accelerometer_bottom_joint
- removed joint left_fr3_link1_accelerometer_top_joint
- removed joint left_fr3_link2_accelerometer_bottom_joint
- removed joint left_fr3_link2_accelerometer_top_joint
- removed joint left_fr3_link3_accelerometer_bottom_joint
- removed joint left_fr3_link3_accelerometer_top_joint
- removed joint left_fr3_link4_accelerometer_bottom_joint
- removed joint left_fr3_link4_accelerometer_top_joint
- removed joint left_fr3_link5_accelerometer_bottom_joint
- removed joint left_fr3_link5_accelerometer_top_joint
- removed joint right_fr3_joint1
- removed joint right_fr3_joint2
- removed joint right_fr3_joint3
- removed joint right_fr3_joint4
- removed joint right_fr3_joint5
- removed joint right_fr3_joint6
- removed joint right_fr3_joint7
- removed joint right_fr3_joint8
- removed joint right_fr3_link0_accelerometer_bottom_joint
- removed joint right_fr3_link0_accelerometer_top_joint
- removed joint right_fr3_link1_accelerometer_bottom_joint
- removed joint right_fr3_link1_accelerometer_top_joint
- removed joint right_fr3_link2_accelerometer_bottom_joint
- removed joint right_fr3_link2_accelerometer_top_joint
- removed joint right_fr3_link3_accelerometer_bottom_joint
- removed joint right_fr3_link3_accelerometer_top_joint
- removed joint right_fr3_link4_accelerometer_bottom_joint
- removed joint right_fr3_link4_accelerometer_top_joint
- removed joint right_fr3_link5_accelerometer_bottom_joint
- removed joint right_fr3_link5_accelerometer_top_joint
- removed joint right_fr3_right_base_joint
- added joint fr3_duo_mount_left_joint: type fixed, parent fr3_duo_mount_origin, child fr3_duo_mount_left, origin xyz=0.0 0.05018 0.0 rpy=-0.89 -0.17 -0.46
- added joint fr3_duo_mount_origin_joint: type fixed, parent fr3_duo_mount_mounting_point, child fr3_duo_mount_origin, origin xyz=0.037 -0.0 0.05 rpy=-0.0 -0.0 -0.0
- added joint fr3_duo_mount_right_joint: type fixed, parent fr3_duo_mount_origin, child fr3_duo_mount_right, origin xyz=0.0 -0.05018 0.0 rpy=0.89 -0.17 0.46
- added joint left_fr3v2_joint1: type revolute, parent left_fr3v2_link0, child left_fr3v2_link1, origin xyz=0 0 0.333 rpy=0 0 0, axis 0 0 1, limit lower=-2.9007400166666666 upper=2.9007400166666666 effort=87.0 velocity=2.62
- added joint left_fr3v2_joint2: type revolute, parent left_fr3v2_link1, child left_fr3v2_link2, origin xyz=0 0 0 rpy=-1.570796326794897 0 0, axis 0 0 1, limit lower=-1.8360900166666667 upper=1.8360900166666667 effort=87.0 velocity=2.62
- added joint left_fr3v2_joint3: type revolute, parent left_fr3v2_link2, child left_fr3v2_link3, origin xyz=0 -0.316 0 rpy=1.570796326794897 0 0, axis 0 0 1, limit lower=-2.9007400166666666 upper=2.9007400166666666 effort=87.0 velocity=2.62
- added joint left_fr3v2_joint4: type revolute, parent left_fr3v2_link3, child left_fr3v2_link4, origin xyz=0.0825 0 0 rpy=1.570796326794897 0 0, axis 0 0 1, limit lower=-3.077020016666667 upper=-0.11693708333333333 effort=87.0 velocity=2.62
- added joint left_fr3v2_joint5: type revolute, parent left_fr3v2_link4, child left_fr3v2_link5, origin xyz=-0.0825 0.384 0 rpy=-1.570796326794897 0 0, axis 0 0 1, limit lower=-2.87630335 upper=2.87630335 effort=12.0 velocity=5.26
- added joint left_fr3v2_joint6: type revolute, parent left_fr3v2_link5, child left_fr3v2_link6, origin xyz=0 0 0 rpy=1.570796326794897 0 0, axis 0 0 1, limit lower=0.43982265 upper=4.62163335 effort=12.0 velocity=4.18
- added joint left_fr3v2_joint7: type revolute, parent left_fr3v2_link6, child left_fr3v2_link7, origin xyz=0.088 0 0 rpy=1.570796326794897 0 0, axis 0 0 1, limit lower=-3.05083335 upper=3.05083335 effort=12.0 velocity=5.26
- added joint left_fr3v2_joint8: type fixed, parent left_fr3v2_link7, child left_fr3v2_link8, origin xyz=0 0 0.107 rpy=0 0 0
- added joint left_fr3v2_left_base_joint: type fixed, parent left_base, child left_fr3v2_link0, origin xyz=0 0 0 rpy=0 0 0
- added joint left_fr3v2_link0_accelerometer_bottom_joint: type fixed, parent left_fr3v2_link0, child left_fr3v2_link0_accelerometer_bottom, origin xyz=-0.019739 0.0015506 0.05075 rpy=0.0 0.0 -1.5708
- added joint left_fr3v2_link0_accelerometer_top_joint: type fixed, parent left_fr3v2_link0, child left_fr3v2_link0_accelerometer_top, origin xyz=-0.017402 -0.007872 0.04715 rpy=3.1416 0.0 0.0
- added joint left_fr3v2_link1_accelerometer_bottom_joint: type fixed, parent left_fr3v2_link1, child left_fr3v2_link1_accelerometer_bottom, origin xyz=0.01974 -0.08975 0.00155 rpy=-1.5708 1.5708 0.0
- added joint left_fr3v2_link1_accelerometer_top_joint: type fixed, parent left_fr3v2_link1, child left_fr3v2_link1_accelerometer_top, origin xyz=0.017402 -0.093352 -0.00787 rpy=-1.5708 0.0 3.1416
- added joint left_fr3v2_link2_accelerometer_bottom_joint: type fixed, parent left_fr3v2_link2, child left_fr3v2_link2_accelerometer_bottom, origin xyz=0.019737 -0.11875 -0.00155 rpy=1.5708 -1.5708 0.0
- added joint left_fr3v2_link2_accelerometer_top_joint: type fixed, parent left_fr3v2_link2, child left_fr3v2_link2_accelerometer_top, origin xyz=0.017403 -0.11515 0.00787 rpy=1.5708 0.0 3.1416
- added joint left_fr3v2_link3_accelerometer_bottom_joint: type fixed, parent left_fr3v2_link3, child left_fr3v2_link3_accelerometer_bottom, origin xyz=0.062769 0.073756 0.00155 rpy=1.5708 1.5708 0.0
- added joint left_fr3v2_link3_accelerometer_top_joint: type fixed, parent left_fr3v2_link3, child left_fr3v2_link3_accelerometer_top, origin xyz=0.065099 0.077352 -0.00787 rpy=-1.5708 0.0 0.0
- added joint left_fr3v2_link4_accelerometer_bottom_joint: type fixed, parent left_fr3v2_link4, child left_fr3v2_link4_accelerometer_bottom, origin xyz=-0.062775 0.049753 0.00155 rpy=-1.5708 1.5708 0.0
- added joint left_fr3v2_link4_accelerometer_top_joint: type fixed, parent left_fr3v2_link4, child left_fr3v2_link4_accelerometer_top, origin xyz=-0.0651 0.046152 -0.00787 rpy=-1.5708 0.0 -3.1416
- added joint left_fr3v2_link5_accelerometer_bottom_joint: type fixed, parent left_fr3v2_link5, child left_fr3v2_link5_accelerometer_bottom, origin xyz=-0.019742 0.082275 0.00146 rpy=1.5708 1.5708 0.0
- added joint left_fr3v2_link5_accelerometer_top_joint: type fixed, parent left_fr3v2_link5, child left_fr3v2_link5_accelerometer_top, origin xyz=-0.017363 0.085872 -0.00795 rpy=-1.5708 0.0 0.0
- added joint right_fr3v2_joint1: type revolute, parent right_fr3v2_link0, child right_fr3v2_link1, origin xyz=0 0 0.333 rpy=0 0 0, axis 0 0 1, limit lower=-2.9007400166666666 upper=2.9007400166666666 effort=87.0 velocity=2.62
- added joint right_fr3v2_joint2: type revolute, parent right_fr3v2_link1, child right_fr3v2_link2, origin xyz=0 0 0 rpy=-1.570796326794897 0 0, axis 0 0 1, limit lower=-1.8360900166666667 upper=1.8360900166666667 effort=87.0 velocity=2.62
- added joint right_fr3v2_joint3: type revolute, parent right_fr3v2_link2, child right_fr3v2_link3, origin xyz=0 -0.316 0 rpy=1.570796326794897 0 0, axis 0 0 1, limit lower=-2.9007400166666666 upper=2.9007400166666666 effort=87.0 velocity=2.62
- added joint right_fr3v2_joint4: type revolute, parent right_fr3v2_link3, child right_fr3v2_link4, origin xyz=0.0825 0 0 rpy=1.570796326794897 0 0, axis 0 0 1, limit lower=-3.077020016666667 upper=-0.11693708333333333 effort=87.0 velocity=2.62
- added joint right_fr3v2_joint5: type revolute, parent right_fr3v2_link4, child right_fr3v2_link5, origin xyz=-0.0825 0.384 0 rpy=-1.570796326794897 0 0, axis 0 0 1, limit lower=-2.87630335 upper=2.87630335 effort=12.0 velocity=5.26
- added joint right_fr3v2_joint6: type revolute, parent right_fr3v2_link5, child right_fr3v2_link6, origin xyz=0 0 0 rpy=1.570796326794897 0 0, axis 0 0 1, limit lower=0.43982265 upper=4.62163335 effort=12.0 velocity=4.18
- added joint right_fr3v2_joint7: type revolute, parent right_fr3v2_link6, child right_fr3v2_link7, origin xyz=0.088 0 0 rpy=1.570796326794897 0 0, axis 0 0 1, limit lower=-3.05083335 upper=3.05083335 effort=12.0 velocity=5.26
- added joint right_fr3v2_joint8: type fixed, parent right_fr3v2_link7, child right_fr3v2_link8, origin xyz=0 0 0.107 rpy=0 0 0
- added joint right_fr3v2_link0_accelerometer_bottom_joint: type fixed, parent right_fr3v2_link0, child right_fr3v2_link0_accelerometer_bottom, origin xyz=-0.019739 0.0015506 0.05075 rpy=0.0 0.0 -1.5708
- added joint right_fr3v2_link0_accelerometer_top_joint: type fixed, parent right_fr3v2_link0, child right_fr3v2_link0_accelerometer_top, origin xyz=-0.017402 -0.007872 0.04715 rpy=3.1416 0.0 0.0
- added joint right_fr3v2_link1_accelerometer_bottom_joint: type fixed, parent right_fr3v2_link1, child right_fr3v2_link1_accelerometer_bottom, origin xyz=0.01974 -0.08975 0.00155 rpy=-1.5708 1.5708 0.0
- added joint right_fr3v2_link1_accelerometer_top_joint: type fixed, parent right_fr3v2_link1, child right_fr3v2_link1_accelerometer_top, origin xyz=0.017402 -0.093352 -0.00787 rpy=-1.5708 0.0 3.1416
- added joint right_fr3v2_link2_accelerometer_bottom_joint: type fixed, parent right_fr3v2_link2, child right_fr3v2_link2_accelerometer_bottom, origin xyz=0.019737 -0.11875 -0.00155 rpy=1.5708 -1.5708 0.0
- added joint right_fr3v2_link2_accelerometer_top_joint: type fixed, parent right_fr3v2_link2, child right_fr3v2_link2_accelerometer_top, origin xyz=0.017403 -0.11515 0.00787 rpy=1.5708 0.0 3.1416
- added joint right_fr3v2_link3_accelerometer_bottom_joint: type fixed, parent right_fr3v2_link3, child right_fr3v2_link3_accelerometer_bottom, origin xyz=0.062769 0.073756 0.00155 rpy=1.5708 1.5708 0.0
- added joint right_fr3v2_link3_accelerometer_top_joint: type fixed, parent right_fr3v2_link3, child right_fr3v2_link3_accelerometer_top, origin xyz=0.065099 0.077352 -0.00787 rpy=-1.5708 0.0 0.0
- added joint right_fr3v2_link4_accelerometer_bottom_joint: type fixed, parent right_fr3v2_link4, child right_fr3v2_link4_accelerometer_bottom, origin xyz=-0.062775 0.049753 0.00155 rpy=-1.5708 1.5708 0.0
- added joint right_fr3v2_link4_accelerometer_top_joint: type fixed, parent right_fr3v2_link4, child right_fr3v2_link4_accelerometer_top, origin xyz=-0.0651 0.046152 -0.00787 rpy=-1.5708 0.0 -3.1416
- added joint right_fr3v2_link5_accelerometer_bottom_joint: type fixed, parent right_fr3v2_link5, child right_fr3v2_link5_accelerometer_bottom, origin xyz=-0.019742 0.082275 0.00146 rpy=1.5708 1.5708 0.0
- added joint right_fr3v2_link5_accelerometer_top_joint: type fixed, parent right_fr3v2_link5, child right_fr3v2_link5_accelerometer_top, origin xyz=-0.017363 0.085872 -0.00795 rpy=-1.5708 0.0 0.0
- added joint right_fr3v2_right_base_joint: type fixed, parent right_base, child right_fr3v2_link0, origin xyz=0 0 0 rpy=0 0 0
- joint left_base_joint: origin xyz=0.0369 0.05018 0.050885 rpy=-0.89334809 -0.17456074 -0.46334506 -> (none); parent mount_link -> fr3_duo_mount_left
- joint mount_joint: child mount_link -> fr3_duo_mount_mounting_point
- joint right_base_joint: origin xyz=0.0369 -0.05018 0.050885 rpy=0.89334809 -0.17456074 0.46334506 -> (none); parent mount_link -> fr3_duo_mount_right
