Commit message: feat: franka vision and manipulation kit sensors displayed in gazebo

File: franka_gazebo_bringup/urdf/mobile_fr3_duo_v0_2_with_sensors.gazebo.urdf.xacro (robot description, xacro)
@@ -6,17 +6,28 @@
          http://www.apache.org/licenses/LICENSE-2.0 -->
 <!--
-  Gazebo entry point for the Mobile FR3 Duo v0.2 with sensors.
-  This file orchestrates the Gazebo simulation:
-    - Instantiates Layer 2 macro (robot + sensor suite)
-    - Applies Gazebo-specific sensor plugins (camera, IMU, LiDAR)
-  Each layer only knows about the layer directly below it:
-    Layer 3 (this file) → Layer 2 macro → Layer 1 macro
+  Gazebo entry point for the Mobile FR3 Duo v0.2 with BOTH sensor suites.
+  ARCHITECTURE: Modular composition from source packages:
+    - Layer 1: Base robot from franka_description
+    - Layer 2a: Mobile platform sensors from franka_mobile_sensors
+    - Layer 2b: Vision kit accessories from franka_vision_and_manipulation_kit
+    - Layer 3: Gazebo plugins applied by franka_gazebo_bringup
+  Result: Robot with 10 sensors fully simulated in Gazebo
+    - 4x RGB cameras (mobile platform) from franka_mobile_sensors
+    - 2x LiDARs (mobile platform) from franka_mobile_sensors
+    - 1x Body IMU (mobile platform) from franka_mobile_sensors
+    - 2x Wrist cameras D405 (vision kit) from franka_vision_and_manipulation_kit
+    - 1x Head camera ZED Mini (vision kit) from franka_vision_and_manipulation_kit
 -->
-<robot xmlns:xacro="http://www.ros.org/wiki/xacro"
-       name="mobile_fr3_duo_v0_2_gazebo_with_sensors">
+<robot xmlns:xacro="http://www.ros.org/wiki/xacro" name="mobile_fr3_duo_v0_2_gazebo_sensors">
   <!-- ================================================================ -->
-  <!-- Macro includes                                                    -->
+  <!-- Includes                                                         -->
   <!-- ================================================================ -->
-  <xacro:include filename="$(find franka_mobile_sensors)/robots/mobile_fr3_duo_v0_2_with_sensors.xacro"/>
+  <!-- Base robot (Layer 1) -->
+  <xacro:include filename="$(find franka_description)/robots/mobile_fr3_duo_v0_2/mobile_fr3_duo_v0_2.xacro"/>
+  <!-- Mobile platform sensor components (Layer 2a) -->
+  <xacro:include filename="$(find franka_mobile_sensors)/robots/sensor_suite.xacro"/>
+  <!-- Vision kit accessory components (Layer 2b) -->
+  <xacro:include filename="$(find franka_vision_and_manipulation_kit)/robots/vision_kit_components.xacro"/>
+  <!-- Gazebo sensor plugins (Layer 3) -->
   <xacro:include filename="$(find franka_gazebo_bringup)/urdf/sensors.xacro" />
   <xacro:include filename="$(find franka_gazebo_bringup)/urdf/gravity_overrides.xacro"/>
@@ -47,7 +58,7 @@
   <xacro:arg name="use_arms"             default="true" />
   <!-- ================================================================ -->
-  <!-- Robot + sensors instantiation (Layer 2 macro)                    -->
+  <!-- LAYER 1: Base Robot                                              -->
   <!-- ================================================================ -->
-  <xacro:mobile_fr3_duo_v0_2_with_sensors
+  <xacro:mobile_fr3_duo_v0_2
         robot_types="$(arg robot_types)"
         hand="$(arg hand)"
@@ -71,29 +82,21 @@
         safety_distance="$(arg safety_distance)"
         with_sc="$(arg with_sc)"/>
-  <!-- ================= CAMERA SENSORS ================= -->
-  <xacro:franka_gazebo_camera link_reference="camera_front_link"
-                              sensor_name="camera_front"
-                              gz_topic="/camera_front/image_raw"/>
-  <xacro:franka_gazebo_camera link_reference="camera_rear_link"
-                              sensor_name="camera_rear"
-                              gz_topic="/camera_rear/image_raw"/>
-  <xacro:franka_gazebo_camera link_reference="camera_left_link"
-                              sensor_name="camera_left"
-                              gz_topic="/camera_left/image_raw"/>
-  <xacro:franka_gazebo_camera link_reference="camera_right_link"
-                              sensor_name="camera_right"
-                              gz_topic="/camera_right/image_raw"/>
-  <!-- ================= LIDAR SENSORS ================= -->
-  <xacro:franka_gazebo_lidar link_reference="lidar_front"
-                              sensor_name="lidar_front"
-                              ros_topic="/lidar_front/scan"/>
-  <xacro:franka_gazebo_lidar link_reference="lidar_rear"
-                              sensor_name="lidar_rear"
-                              ros_topic="/lidar_rear/scan"/>
-  <!-- ================= IMU SENSOR ================= -->
-  <xacro:franka_gazebo_body_imu link_reference="imu_body_link"
-                                gz_topic="/imu/data"/>
   <!-- ================================================================ -->
-  <!-- Gravity overrides                                                -->
+  <!-- LAYER 2a: Mobile Platform Sensors                               -->
+  <!-- ================================================================ -->
+  <xacro:sensor_suite />
+  <!-- ================================================================ -->
+  <!-- LAYER 2b: Vision Kit Accessories                                -->
+  <!-- ================================================================ -->
+  <xacro:vision_kit_components left_arm_type="fr3v2" right_arm_type="fr3v2" prefix="" robotiq_use_fake_hardware="true" robotiq_include_ros2_control="true" sim_gazebo="true" />
+  <!-- ================================================================ -->
+  <!-- LAYER 3: Gazebo Sensor Plugins                                  -->
+  <!-- ================================================================ -->
+  <!-- Mobile Platform Sensors (4x D455 RGB, 2x LiDAR, 1x IMU) -->
+  <xacro:franka_gazebo_mobile_platform_sensors/>
+  <!-- Vision Kit Sensors (2x D405 wrist, 1x ZED head) -->
+  <xacro:franka_gazebo_vision_kit_sensors/>
+  <!-- ================================================================ -->
+  <!-- Physics Configuration                                            -->
   <!-- ================================================================ -->
   <xacro:disable_arm_gravity prefix="left_" robot_type="${robot_types_list[1]}"/>

File: franka_gazebo_bringup/urdf/sensors.xacro (robot description, xacro)
@@ -118,3 +118,99 @@
         </gazebo>
     </xacro:macro>
+    <!-- ================= D405 REALSENSE CAMERA MACRO ================= -->
+    <xacro:macro name="franka_gazebo_d405" params="link_reference sensor_name gz_topic
+                 rate:=30 hfov:=1.047 width:=640 height:=480 format:=R8G8B8
+                 clip_near:=0.1 clip_far:=100.0 visualize:=true">
+        <gazebo reference="${link_reference}">
+            <sensor name="${sensor_name}" type="camera">
+                <pose>0 0 0 0 0 0</pose>
+                <topic>${gz_topic}</topic>
+                <update_rate>${rate}</update_rate>
+                <camera>
+                    <horizontal_fov>${hfov}</horizontal_fov>
+                    <image>
+                        <width>${width}</width>
+                        <height>${height}</height>
+                        <format>${format}</format>
+                    </image>
+                    <clip>
+                        <near>${clip_near}</near>
+                        <far>${clip_far}</far>
+                    </clip>
+                </camera>
+                <always_on>true</always_on>
+                <visualize>${visualize}</visualize>
+            </sensor>
+        </gazebo>
+    </xacro:macro>
+    <!-- ================= ZED CAMERA MACRO ================= -->
+    <xacro:macro name="franka_gazebo_zed" params="link_reference sensor_name gz_topic
+                 rate:=30 hfov:=1.5708 width:=672 height:=376 format:=R8G8B8
+                 clip_near:=0.1 clip_far:=100.0 visualize:=true">
+        <gazebo reference="${link_reference}">
+            <sensor name="${sensor_name}" type="camera">
+                <pose>0 0 0 0 0 0</pose>
+                <topic>${gz_topic}</topic>
+                <update_rate>${rate}</update_rate>
+                <camera>
+                    <horizontal_fov>${hfov}</horizontal_fov>
+                    <image>
+                        <width>${width}</width>
+                        <height>${height}</height>
+                        <format>${format}</format>
+                    </image>
+                    <clip>
+                        <near>${clip_near}</near>
+                        <far>${clip_far}</far>
+                    </clip>
+                </camera>
+                <always_on>true</always_on>
+                <visualize>${visualize}</visualize>
+            </sensor>
+        </gazebo>
+    </xacro:macro>
+    <!-- ================= CONVENIENCE MACROS FOR FUTURE VARIANTS ================= -->
+    <!-- These macros provide reusable groups for common sensor configurations      -->
+    <!-- Allows easy composition for future variants (e.g., FR3 Duo only)           -->
+    <!-- All mobile platform sensors (RGB cameras, LiDARs, IMU) -->
+    <xacro:macro name="franka_gazebo_mobile_platform_sensors">
+        <xacro:franka_gazebo_camera link_reference="camera_front_link"
+                                    sensor_name="camera_front"
+                                    gz_topic="/camera_front/image_raw"/>
+        <xacro:franka_gazebo_camera link_reference="camera_rear_link"
+                                    sensor_name="camera_rear"
+                                    gz_topic="/camera_rear/image_raw"/>
+        <xacro:franka_gazebo_camera link_reference="camera_left_link"
+                                    sensor_name="camera_left"
+                                    gz_topic="/camera_left/image_raw"/>
+        <xacro:franka_gazebo_camera link_reference="camera_right_link"
+                                    sensor_name="camera_right"
+                                    gz_topic="/camera_right/image_raw"/>
+        <xacro:franka_gazebo_lidar link_reference="lidar_front"
+                                    sensor_name="lidar_front"
+                                    ros_topic="/lidar_front/scan"/>
+        <xacro:franka_gazebo_lidar link_reference="lidar_rear"
+                                    sensor_name="lidar_rear"
+                                    ros_topic="/lidar_rear/scan"/>
+        <xacro:franka_gazebo_body_imu link_reference="imu_body_link"
+                                      gz_topic="/imu/data"/>
+    </xacro:macro>
+    <!-- All vision and manipulation kit sensors (wrist D405 + head ZED) -->
+    <xacro:macro name="franka_gazebo_vision_kit_sensors">
+        <xacro:franka_gazebo_d405
+            link_reference="left__wrist_camera_link"
+            sensor_name="left_wrist_camera"
+            gz_topic="/left_wrist_camera/image_raw"
+            width="640" height="480" />
+        <xacro:franka_gazebo_d405
+            link_reference="right__wrist_camera_link"
+            sensor_name="right_wrist_camera"
+            gz_topic="/right_wrist_camera/image_raw"
+            width="640" height="480" />
+        <xacro:franka_gazebo_zed
+            link_reference="head_camera_link"
+            sensor_name="head_camera"
+            gz_topic="/head_camera/image_raw"
+            width="672" height="376" />
+    </xacro:macro>
 </robot>

File: franka_vision_and_manipulation_kit/accessories/robotiq_gripper_with_realsense_camera.xacro (robot description, xacro)
@@ -12,9 +12,9 @@
       robotiq_adapter_rotation:=^|${-pi/2}
       robotiq_name:=RobotiqGripperHardwareInterface
-      robotiq_com_port:='/dev/ttyUSB0'
+      robotiq_com_port:=/dev/ttyUSB0
       robotiq_sim_isaac:=false
+      robotiq_sim_gazebo:=false
       robotiq_use_fake_hardware:=false
       robotiq_include_ros2_control:=true
-      robotiq_com_port:=/dev/ttyUSB0
       realsense_use_nominal_extrinsics:=true
       ">
@@ -27,4 +27,5 @@
         parent="${prefix}gripper_mount_link"
         com_port="${robotiq_com_port}"
+        sim_gazebo="${robotiq_sim_gazebo}"
         sim_isaac="${robotiq_sim_isaac}"
         use_fake_hardware="${robotiq_use_fake_hardware}"

File: franka_vision_and_manipulation_kit/robots/vision_and_manipulation_kit.xacro (robot description, xacro)
@@ -4,6 +4,5 @@
   <xacro:include filename="$(find franka_description)/accessories/franka_head_v0_2/franka_head.xacro"/>
   <xacro:include filename="$(find franka_description)/robots/mobile_fr3_duo_v0_2/mobile_fr3_duo_v0_2.xacro" />
-  <xacro:include filename="$(find zed_description)/urdf/zed_macro.urdf.xacro"/>
-  <xacro:include filename="$(find franka_vision_and_manipulation_kit)/accessories/robotiq_gripper_with_realsense_camera.xacro" />
+  <xacro:include filename="$(find franka_vision_and_manipulation_kit)/robots/vision_kit_components.xacro" />
   <xacro:macro name="fr3_duo_with_vision_and_manipulation_kit"
     params="
@@ -94,14 +93,6 @@
         with_sc="$(arg with_sc)" />
     </xacro:unless>
-    <xacro:robotiq_gripper_with_realsense_camera parent="left_$(arg left_arm_type)_link8" prefix="$(arg prefix)left_" />
-    <xacro:robotiq_gripper_with_realsense_camera parent="right_$(arg right_arm_type)_link8" prefix="$(arg prefix)right_" />
-    <xacro:zed_camera name="$(arg prefix)head" model="zedm" custom_baseline="0.0" enable_gnss="false">
-        <origin xyz="0.0 0.0 0.0" rpy="0 0 0"/>
-    </xacro:zed_camera>
-    <joint name="$(arg prefix)head_camera_mounting_point_to_head_camera_link" type="fixed">
-      <parent link="$(arg prefix)head_camera_mounting_point"/>
-      <child link="$(arg prefix)head_camera_link"/>
-      <origin xyz="0.0015 -0.011 -0.013" rpy="0 0 0"/>
-    </joint>
+    <!-- Attach vision kit components (wrist cameras + head camera) -->
+    <xacro:vision_kit_components left_arm_type="$(arg left_arm_type)" right_arm_type="$(arg right_arm_type)" prefix="$(arg prefix)" robotiq_use_fake_hardware="$(arg use_fake_hardware)" robotiq_include_ros2_control="$(arg ros2_control)" />
   </xacro:macro>
 </robot>
