Commit message: refactor: Migrating ros2_control content from franka_description to franka_hardware

File: franka_gazebo_bringup/urdf/fr3_duo.gazebo.urdf.xacro (robot description, xacro)
@@ -17,10 +17,9 @@
   <xacro:include filename="$(find franka_description)/robots/fr3_duo/fr3_duo.xacro"/>
   <xacro:include filename="$(find franka_gazebo_bringup)/urdf/gravity_overrides.xacro"/>
+  <!-- Unified ros2_control for gazebo (both arms in one block) -->
+  <xacro:include filename="$(find franka_hardware)/ros2_control/fr3_duo.ros2_control.xacro"/>
   <!-- ================================================================ -->
   <!-- Arguments                                                        -->
   <!-- ================================================================ -->
-  <!-- For Gazebo, ros2_control must be false on individual robots,
-       with a single unified ros2_control block instead -->
-  <xacro:property name="ros_control_flag" value="false"/>
   <xacro:arg name="robot_types" default="['fr3v2','fr3v2']" />
   <xacro:property name="robot_types_list" value="${$(arg robot_types)}" />
@@ -37,9 +36,4 @@
   <xacro:arg name="safety_distance"    default="0.03" />
   <xacro:arg name="with_sc"            default="false" />
-  <xacro:arg name="ros2_control"       default="true" />
-  <xacro:arg name="robot_ips"          default="['172.16.0.1','172.16.0.2']" />
-  <xacro:property name="robot_ips_list" value="${$(arg robot_ips)}" />
-  <xacro:arg name="use_fake_hardware"    default="false" />
-  <xacro:arg name="fake_sensor_commands" default="false" />
   <xacro:arg name="gazebo_effort"        default="false" />
   <xacro:arg name="description_pkg"      default="franka_description" />
@@ -58,10 +52,5 @@
         arm_prefixes="${arm_prefixes_list}"
         hand="$(arg hand)"
-        ros2_control="${ros_control_flag}"
         gazebo="true"
-        gazebo_effort="$(arg gazebo_effort)"
-        use_fake_hardware="$(arg use_fake_hardware)"
-        fake_sensor_commands="$(arg fake_sensor_commands)"
-        robot_ips="$(arg robot_ips)"
         description_pkg="$(arg description_pkg)"
         base_mount="$(arg base_mount)"
@@ -76,4 +65,11 @@
         safety_distance="$(arg safety_distance)"
         with_sc="$(arg with_sc)"/>
+  <!-- Unified ros2_control for both arms (gazebo mode) -->
+  <xacro:fr3_duo_ros2_control
+        robot_types="${robot_types_list}"
+        arm_prefixes="${arm_prefixes_list}"
+        hand="$(arg hand)"
+        gazebo="true"
+        gazebo_effort="$(arg gazebo_effort)"/>
   <!-- ================================================================ -->
   <!-- Gravity overrides                                                -->

File: franka_gazebo_bringup/urdf/fr3_duo_with_sensors.gazebo.urdf.xacro (robot description, xacro)
@@ -23,4 +23,6 @@
   <!-- Vision kit accessory components (Layer 2b) -->
   <xacro:include filename="$(find franka_vision_and_manipulation_kit)/robots/vision_kit_components.xacro"/>
+  <!-- ros2_control hardware interface (unified for both arms in gazebo) -->
+  <xacro:include filename="$(find franka_hardware)/ros2_control/fr3_duo.ros2_control.xacro"/>
   <!-- Gazebo sensor plugins (Layer 3) -->
   <xacro:include filename="$(find franka_gazebo_bringup)/urdf/sensors.xacro" />
@@ -43,14 +45,8 @@
   <xacro:arg name="safety_distance"    default="0.03" />
   <xacro:arg name="with_sc"            default="false" />
-  <xacro:arg name="robot_ips"          default="['172.16.0.1','172.16.0.2']" />
-  <xacro:property name="robot_ips_list" value="${$(arg robot_ips)}" />
-  <xacro:arg name="use_fake_hardware"    default="false" />
-  <xacro:arg name="fake_sensor_commands" default="false" />
   <xacro:arg name="gazebo_effort"        default="false" />
   <xacro:arg name="description_pkg"      default="franka_description" />
   <xacro:arg name="base_mount"           default="world"/>
   <xacro:arg name="connected_to"         default="world"/>
-  <!-- For Gazebo simulation, disable ros2_control in fr3_duo macro -->
-  <xacro:property name="ros_control_flag" value="false"/>
   <!-- ================================================================ -->
   <!-- World link definition                                            -->
@@ -65,10 +61,5 @@
         arm_prefixes="${arm_prefixes_list}"
         hand="$(arg hand)"
-        ros2_control="${ros_control_flag}"
         gazebo="true"
-        gazebo_effort="$(arg gazebo_effort)"
-        use_fake_hardware="$(arg use_fake_hardware)"
-        fake_sensor_commands="$(arg fake_sensor_commands)"
-        robot_ips="$(arg robot_ips)"
         description_pkg="$(arg description_pkg)"
         base_mount="$(arg base_mount)"
@@ -88,4 +79,13 @@
   <xacro:vision_kit_components left_arm_type="fr3v2" right_arm_type="fr3v2" prefix="" robotiq_use_fake_hardware="true" robotiq_include_ros2_control="true" sim_gazebo="true" />
   <!-- ================================================================ -->
+  <!-- ros2_control: Unified for both arms (gazebo mode)               -->
+  <!-- ================================================================ -->
+  <xacro:fr3_duo_ros2_control
+        robot_types="${robot_types_list}"
+        arm_prefixes="${arm_prefixes_list}"
+        hand="$(arg hand)"
+        gazebo="true"
+        gazebo_effort="$(arg gazebo_effort)"/>
+  <!-- ================================================================ -->
   <!-- LAYER 3: Gazebo Sensor Plugins                                  -->
   <!-- ================================================================ -->

File: franka_gazebo_bringup/urdf/franka_arm.gazebo.xacro (robot description, xacro)
@@ -1,12 +1,43 @@
 <?xml version="1.0" encoding="utf-8"?>
+<!--
+  Gazebo entry point for single-arm (FR3/FP3/FER).
+  Includes the franka_description base robot, ros2_control hardware interface,
+  Gazebo-specific sensors, and gravity overrides.
+-->
 <robot xmlns:xacro="http://www.ros.org/wiki/xacro" name="$(arg robot_type)">
+    <!-- ================================================================ -->
+    <!-- Macro includes                                                    -->
+    <!-- ================================================================ -->
     <xacro:arg name="robot_type" default="fr3"/>
-    <!-- Include base robot fr3 -->
+    <!-- Base robot (Layer 1) -->
     <xacro:include filename="$(find franka_description)/robots/$(arg robot_type)/$(arg robot_type).urdf.xacro"/>
-    <!-- Include gazebo macros -->
+    <!-- ros2_control hardware interface -->
+    <xacro:include filename="$(find franka_hardware)/ros2_control/franka_arm.ros2_control.xacro"/>
+    <!-- Gazebo extras -->
     <xacro:include filename="$(find franka_gazebo_bringup)/urdf/sensors.xacro"/>
     <xacro:include filename="$(find franka_gazebo_bringup)/urdf/gravity_overrides.xacro"/>
+    <!-- ================================================================ -->
+    <!-- Arguments                                                        -->
+    <!-- ================================================================ -->
+    <xacro:arg name="arm_prefix" default=""/>
+    <xacro:arg name="hand" default="true"/>
+    <xacro:arg name="ee_id" default="franka_hand"/>
+    <xacro:arg name="gazebo_effort" default="false"/>
+    <!-- Compute prefix (same logic as fr3.urdf.xacro) -->
+    <xacro:property name="prefix" value="$(arg arm_prefix)"/>
+    <xacro:property name="modified_prefix" value="${prefix + '_' if prefix else ''}"/>
+    <!-- ================================================================ -->
+    <!-- ros2_control hardware interface (gazebo mode)                    -->
+    <!-- ================================================================ -->
+    <xacro:franka_arm_ros2_control
+        robot_type="$(arg robot_type)"
+        gazebo="true"
+        hand="$(arg hand)"
+        gazebo_effort="$(arg gazebo_effort)"
+        arm_prefix="${modified_prefix}"/>
+    <!-- ================================================================ -->
+    <!-- Gazebo sensors and physics overrides                             -->
+    <!-- ================================================================ -->
     <!-- Arm IMUs -->
-    <!-- arm prefix is inherited from the franka_description xacro -->
     <xacro:franka_gazebo_arm_imus arm_prefix="$(arg arm_prefix)" robot_type="$(arg robot_type)" imu_side="top"/>
     <xacro:franka_gazebo_arm_imus arm_prefix="$(arg arm_prefix)" robot_type="$(arg robot_type)" imu_side="bottom"/>

File: franka_gazebo_bringup/urdf/mobile_fr3_duo_v0_2.gazebo.urdf.xacro (robot description, xacro)
@@ -17,4 +17,6 @@
   <xacro:include filename="$(find franka_description)/robots/mobile_fr3_duo_v0_2/mobile_fr3_duo_v0_2.xacro"/>
   <xacro:include filename="$(find franka_gazebo_bringup)/urdf/gravity_overrides.xacro"/>
+  <!-- Unified ros2_control for gazebo (mobile base + both arms in one block) -->
+  <xacro:include filename="$(find franka_hardware)/ros2_control/mobile_fr3_duo.ros2_control.xacro"/>
   <!-- ================================================================ -->
   <!-- Arguments                                                        -->
@@ -32,9 +34,4 @@
   <xacro:arg name="safety_distance"    default="0.03" />
   <xacro:arg name="with_sc"            default="false" />
-  <xacro:arg name="ros2_control"       default="false" />
-  <xacro:arg name="robot_ips"          default="['172.16.0.1','172.16.0.2','172.16.0.3']" />
-  <xacro:property name="robot_ips_list" value="${$(arg robot_ips)}" />
-  <xacro:arg name="use_fake_hardware"    default="false" />
-  <xacro:arg name="fake_sensor_commands" default="false" />
   <xacro:arg name="gazebo_effort"        default="false" />
   <xacro:arg name="description_pkg"      default="franka_description" />
@@ -48,11 +45,6 @@
         robot_types="$(arg robot_types)"
         hand="$(arg hand)"
-        ros2_control="$(arg ros2_control)"
         gazebo="true"
-        gazebo_effort="$(arg gazebo_effort)"
-        use_fake_hardware="$(arg use_fake_hardware)"
-        fake_sensor_commands="$(arg fake_sensor_commands)"
         reduced_version="$(arg reduced_version)"
-        robot_ips="$(arg robot_ips)"
         description_pkg="$(arg description_pkg)"
         connected_to="$(arg connected_to)"
@@ -67,4 +59,14 @@
         safety_distance="$(arg safety_distance)"
         with_sc="$(arg with_sc)"/>
+  <!-- Unified ros2_control for gazebo (mobile base + both arms) -->
+  <xacro:property name="arm_prefixes_list" value="${['left','right']}"/>
+  <xacro:mobile_fr3_duo_ros2_control
+        mobile_robot_type="tmrv0_2"
+        robot_types="${robot_types_list}"
+        arm_prefixes="${arm_prefixes_list}"
+        hand="$(arg hand)"
+        gazebo="true"
+        gazebo_effort="$(arg gazebo_effort)"
+        robot_namespace=""/>
   <!-- ================================================================ -->
   <!-- Gravity overrides                                                -->

File: franka_gazebo_bringup/urdf/mobile_fr3_duo_v0_2_with_sensors.gazebo.urdf.xacro (robot description, xacro)
@@ -29,4 +29,6 @@
   <!-- Vision kit accessory components (Layer 2b) -->
   <xacro:include filename="$(find franka_vision_and_manipulation_kit)/robots/vision_kit_components.xacro"/>
+  <!-- ros2_control hardware interface macros -->
+  <xacro:include filename="$(find franka_hardware)/ros2_control/mobile_fr3_duo.ros2_control.xacro"/>
   <!-- Gazebo sensor plugins (Layer 3) -->
   <xacro:include filename="$(find franka_gazebo_bringup)/urdf/sensors.xacro" />
@@ -47,14 +49,9 @@
   <xacro:arg name="safety_distance"    default="0.03" />
   <xacro:arg name="with_sc"            default="false" />
-  <xacro:arg name="ros2_control"       default="false" />
-  <xacro:arg name="robot_ips"          default="['172.16.0.1','172.16.0.2','172.16.0.3']" />
-  <xacro:property name="robot_ips_list" value="${$(arg robot_ips)}" />
-  <xacro:arg name="use_fake_hardware"    default="false" />
-  <xacro:arg name="fake_sensor_commands" default="false" />
-  <xacro:arg name="gazebo_effort"        default="false" />
   <xacro:arg name="description_pkg"      default="franka_description" />
   <xacro:arg name="connected_to"         default="base" />
   <xacro:arg name="reduced_version"      default="false" />
   <xacro:arg name="use_arms"             default="true" />
+  <xacro:arg name="gazebo_effort"        default="false" />
   <!-- ================================================================ -->
   <!-- LAYER 1: Base Robot                                              -->
@@ -63,11 +60,6 @@
         robot_types="$(arg robot_types)"
         hand="$(arg hand)"
-        ros2_control="$(arg ros2_control)"
         gazebo="true"
-        gazebo_effort="$(arg gazebo_effort)"
-        use_fake_hardware="$(arg use_fake_hardware)"
-        fake_sensor_commands="$(arg fake_sensor_commands)"
         reduced_version="$(arg reduced_version)"
-        robot_ips="$(arg robot_ips)"
         description_pkg="$(arg description_pkg)"
         connected_to="$(arg connected_to)"
@@ -91,4 +83,16 @@
   <xacro:vision_kit_components left_arm_type="fr3v2" right_arm_type="fr3v2" prefix="" robotiq_use_fake_hardware="true" robotiq_include_ros2_control="true" sim_gazebo="true" />
   <!-- ================================================================ -->
+  <!-- ros2_control: Unified mobile base + both arms                   -->
+  <!-- ================================================================ -->
+  <xacro:property name="arm_prefixes_list" value="${['left','right']}"/>
+  <xacro:mobile_fr3_duo_ros2_control
+        mobile_robot_type="tmrv0_2"
+        robot_types="${robot_types_list}"
+        arm_prefixes="${arm_prefixes_list}"
+        hand="$(arg hand)"
+        gazebo="true"
+        gazebo_effort="$(arg gazebo_effort)"
+        robot_namespace=""/>
+  <!-- ================================================================ -->
   <!-- LAYER 3: Gazebo Sensor Plugins                                  -->
   <!-- ================================================================ -->

File: franka_mobile_fr3_duo_moveit_config/urdf/mobile_fr3_duo_v0_2.moveit.urdf.xacro (robot description, xacro)
@@ -8,4 +8,7 @@
        name="mobile_fr3_duo_v0_2">
     <xacro:include filename="$(find franka_description)/robots/mobile_fr3_duo_v0_2/mobile_fr3_duo_v0_2.xacro"/>
+    <!-- ros2_control hardware interface macros -->
+    <xacro:include filename="$(find franka_hardware)/ros2_control/franka_arm.ros2_control.xacro"/>
+    <xacro:include filename="$(find franka_hardware)/ros2_control/tmrv0_2.ros2_control.xacro"/>
     <xacro:arg name="robot_ips"          default="['172.16.16.10', '172.16.16.12', '172.16.16.11']" />
     <xacro:arg name="robot_types" default="['tmrv0_2','fr3v2','fr3v2']" />
@@ -13,5 +16,4 @@
     <xacro:arg name="hand"               default="false" />
     <xacro:arg name="ee_id"              default="None" />
-    <xacro:arg name="ros2_control"       default="true" />
     <xacro:property name="robot_ips_list" value="${$(arg robot_ips)}" />
     <xacro:arg name="gazebo_effort"        default="false" />
@@ -96,15 +98,8 @@
     </joint>
     <xacro:mobile_fr3_duo_v0_2
-        robot_ips="$(arg robot_ips)"
         robot_types="$(arg robot_types)"
         hand="$(arg hand)"
         ee_id="$(arg ee_id)"
-        ros2_control="$(arg ros2_control)"
         gazebo="$(arg gazebo)"
-        gazebo_effort="$(arg gazebo_effort)"
-        use_fake_hardware="$(arg use_fake_hardware)"
-        is_async="$(arg is_async)"
-        thread_priority="$(arg thread_priority)"
-        fake_sensor_commands="$(arg fake_sensor_commands)"
         reduced_version="$(arg reduced_version)"
         description_pkg="$(arg description_pkg)"
@@ -120,4 +115,39 @@
         with_sc="$(arg with_sc)"
     />
+    <!-- ros2_control hardware interfaces -->
+    <xacro:property name="arm_prefixes_list" value="${['left','right']}"/>
+    <!-- TMR mobile base ros2_control -->
+    <xacro:tmrv0_2_ros2_control
+        mobile_robot_type="${robot_types_list[0]}"
+        robot_ip="${robot_ips_list[0]}"
+        use_fake_hardware="$(arg use_fake_hardware)"
+        fake_sensor_commands="$(arg fake_sensor_commands)"
+        gazebo="$(arg gazebo)"
+        robot_namespace=""
+        is_async="$(arg is_async)"
+        thread_priority="$(arg thread_priority)"/>
+    <!-- Per-arm ros2_control -->
+    <xacro:franka_arm_ros2_control
+        robot_type="${robot_types_list[1]}"
+        robot_ip="${robot_ips_list[1]}"
+        use_fake_hardware="$(arg use_fake_hardware)"
+        fake_sensor_commands="$(arg fake_sensor_commands)"
+        gazebo="$(arg gazebo)"
+        hand="$(arg hand)"
+        gazebo_effort="$(arg gazebo_effort)"
+        arm_prefix="${arm_prefixes_list[0]}_"
+        is_async="$(arg is_async)"
+        thread_priority="$(arg thread_priority)"/>
+    <xacro:franka_arm_ros2_control
+        robot_type="${robot_types_list[2]}"
+        robot_ip="${robot_ips_list[2]}"
+        use_fake_hardware="$(arg use_fake_hardware)"
+        fake_sensor_commands="$(arg fake_sensor_commands)"
+        gazebo="$(arg gazebo)"
+        hand="$(arg hand)"
+        gazebo_effort="$(arg gazebo_effort)"
+        arm_prefix="${arm_prefixes_list[1]}_"
+        is_async="$(arg is_async)"
+        thread_priority="$(arg thread_priority)"/>
     <xacro:if value="$(arg gazebo)">
         <xacro:include filename="$(find franka_gazebo_bringup)/urdf/gravity_overrides.xacro"/>

File: franka_mobile_sensors/robots/mobile_fr3_duo_v0_2_with_sensors.urdf.xacro (robot description, xacro)
@@ -25,17 +25,6 @@
   <!-- Should self-collision be enabled? -->
   <xacro:arg name="with_sc" default="false" />
-  <!-- Is the robot being controlled with ros2_control? -->
-  <xacro:arg name="ros2_control" default="false" />
-  <!-- IP address or hostname of the robot -->
-  <xacro:arg name="robot_ips" default="['172.16.0.1','172.16.0.2','172.16.0.3']" />
-  <xacro:property name="robot_ips_list" value="${$(arg robot_ips)}" />
-  <!-- Should a fake hardware be used? -->
-  <xacro:arg name="use_fake_hardware" default="false" />
-  <!-- Should fake sensors be used? -->
-  <xacro:arg name="fake_sensor_commands" default="false" />
   <!-- Should the robot be spawned in Gazebo? -->
   <xacro:arg name="gazebo" default="false" />
-  <!-- Should the robot be spawned in Gazebo with effort interfaces? -->
-  <xacro:arg name="gazebo_effort" default="false" />
   <!-- Name of the description package -->
   <xacro:arg name="description_pkg" default="franka_description" />
@@ -57,11 +46,6 @@
         robot_types="$(arg robot_types)"
         hand="$(arg hand)"
-        ros2_control="$(arg ros2_control)"
         gazebo="$(arg gazebo)"
-        gazebo_effort="$(arg gazebo_effort)"
-        use_fake_hardware="$(arg use_fake_hardware)"
-        fake_sensor_commands="$(arg fake_sensor_commands)"
         reduced_version="$(arg reduced_version)"
-        robot_ips="$(arg robot_ips)"
         description_pkg="$(arg description_pkg)"
         connected_to="$(arg connected_to)"

File: franka_mobile_sensors/robots/mobile_fr3_duo_v0_2_with_sensors.xacro (robot description, xacro)
@@ -25,10 +25,5 @@
               safety_distance
               with_sc
-              ros2_control
-              robot_ips
-              use_fake_hardware
-              fake_sensor_commands
               gazebo
-              gazebo_effort
               description_pkg
               connected_to
@@ -39,11 +34,6 @@
           robot_types="${robot_types}"
           hand="${hand}"
-          ros2_control="${ros2_control}"
           gazebo="${gazebo}"
-          gazebo_effort="${gazebo_effort}"
-          use_fake_hardware="${use_fake_hardware}"
-          fake_sensor_commands="${fake_sensor_commands}"
           reduced_version="${reduced_version}"
-          robot_ips="${robot_ips}"
           description_pkg="${description_pkg}"
           connected_to="${connected_to}"

File: franka_mobile_sensors/robots/tmrv0_2_with_sensors.urdf.xacro (robot description, xacro)
@@ -4,12 +4,4 @@
   <!-- The ID of the robot model to be used -->
   <xacro:arg name="robot_type" default="tmrv0_2" />
-  <!-- Is the robot being controlled with ros2_control? -->
-  <xacro:arg name="ros2_control" default="false" />
-  <!-- IP address or hostname of the robot -->
-  <xacro:arg name="robot_ip" default="172.16.0.4" />
-  <!-- Should a fake hardware be used? -->
-  <xacro:arg name="use_fake_hardware" default="false" />
-  <!-- Should fake sensors be used? -->
-  <xacro:arg name="fake_sensor_commands" default="false" />
   <!-- Should the reduced kinematic version (without caster wheels) be used? -->
   <xacro:arg name="reduced_version" default="false" />
@@ -28,8 +20,4 @@
   <xacro:tmrv0_2_with_sensors
             robot_type="$(arg robot_type)"
-            robot_ip="$(arg robot_ip)"
-            ros2_control="$(arg ros2_control)"
-            use_fake_hardware="$(arg use_fake_hardware)"
-            fake_sensor_commands="$(arg fake_sensor_commands)"
             reduced_version="$(arg reduced_version)"
             robot_namespace="$(arg robot_namespace)"

File: franka_mobile_sensors/robots/tmrv0_2_with_sensors.xacro (robot description, xacro)
@@ -11,8 +11,4 @@
   <xacro:macro name="tmrv0_2_with_sensors"
       params="robot_type
-              ros2_control
-              robot_ip
-              use_fake_hardware
-              fake_sensor_commands
               reduced_version
               gazebo
@@ -20,8 +16,4 @@
     <!-- Instantiate the base robot (Layer 1) -->
     <xacro:tmrv0_2 mobile_robot_type="${robot_type}"
-                robot_ip="${robot_ip}"
-                ros2_control="${ros2_control}"
-                use_fake_hardware="${use_fake_hardware}"
-                fake_sensor_commands="${fake_sensor_commands}"
                 reduced_version="${reduced_version}"
                 robot_namespace="${robot_namespace}"

File: franka_vision_and_manipulation_kit/robots/vision_and_manipulation_kit.xacro (robot description, xacro)
@@ -37,5 +37,4 @@
         robot_types="${['$(arg left_arm_type)', '$(arg right_arm_type)']}"
         arm_prefixes="${['$(arg prefix)left', '$(arg prefix)right']}"
-        robot_ips="${['$(arg left_arm_ip)', '$(arg right_arm_ip)']}"
         hand="false"
         ee_id="none"
@@ -48,9 +47,5 @@
         safety_distance="$(arg safety_distance)"
         with_sc="$(arg with_sc)"
-        ros2_control="$(arg ros2_control)"
-        use_fake_hardware="$(arg use_fake_hardware)"
-        fake_sensor_commands="$(arg fake_sensor_commands)"
         gazebo="$(arg gazebo)"
-        gazebo_effort="$(arg gazebo_effort)"
         description_pkg="$(arg description_pkg)"
         connected_to=""
@@ -73,11 +68,6 @@
         robot_types="${robot_types_list}"
         hand="false"
-        ros2_control="$(arg ros2_control)"
         gazebo="$(arg gazebo)"
-        gazebo_effort="$(arg gazebo_effort)"
-        use_fake_hardware="$(arg use_fake_hardware)"
-        fake_sensor_commands="$(arg fake_sensor_commands)"
         reduced_version="false"
-        robot_ips="${robot_ips_list}"
         description_pkg="$(arg description_pkg)"
         connected_to="base"
