Commit message: refactor: Backport from jazzy about moving ros2_control content to franka_hardware

File: franka_gazebo_bringup/urdf/franka_arm.gazebo.xacro (robot description, xacro)
@@ -1,8 +1,42 @@
 <?xml version="1.0" encoding="utf-8"?>
+<!--
+  Gazebo entry point for single-arm (FR3/FP3/FER).
+  Includes the franka_description base robot, ros2_control hardware interface,
+  and Gazebo-specific sensors.
+-->
 <robot xmlns:xacro="http://www.ros.org/wiki/xacro" name="$(arg robot_type)">
+    <!-- ================================================================ -->
+    <!-- Macro includes                                                    -->
+    <!-- ================================================================ -->
     <xacro:arg name="robot_type" default="fr3"/>
-    <!-- Include base robot fr3 -->
+    <!-- Base robot (Layer 1) -->
     <xacro:include filename="$(find franka_description)/robots/$(arg robot_type)/$(arg robot_type).urdf.xacro"/>
+    <!-- ros2_control hardware interface -->
+    <xacro:include filename="$(find franka_hardware)/ros2_control/franka_arm.ros2_control.xacro"/>
+    <!-- Gazebo extras -->
     <xacro:include filename="$(find franka_gazebo_bringup)/urdf/sensors.xacro"/>
+    <!-- ================================================================ -->
+    <!-- Arguments                                                        -->
+    <!-- ================================================================ -->
+    <xacro:arg name="arm_prefix" default=""/>
+    <xacro:arg name="hand" default="true"/>
+    <xacro:arg name="ee_id" default="franka_hand"/>
+    <xacro:arg name="gazebo_effort" default="false"/>
+    <!-- Compute prefix (same logic as fr3.urdf.xacro) -->
+    <xacro:property name="prefix" value="$(arg arm_prefix)"/>
+    <xacro:property name="modified_prefix" value="${prefix + '_' if prefix else ''}"/>
+    <!-- ================================================================ -->
+    <!-- ros2_control hardware interface (gazebo mode)                    -->
+    <!-- ================================================================ -->
+    <xacro:franka_arm_ros2_control
+        robot_type="$(arg robot_type)"
+        gazebo="true"
+        hand="$(arg hand)"
+        gazebo_effort="$(arg gazebo_effort)"
+        arm_prefix="${modified_prefix}"/>
+    <!-- ================================================================ -->
+    <!-- Gazebo sensors                                                    -->
+    <!-- ================================================================ -->
+    <!-- Arm IMUs -->
     <xacro:franka_gazebo_arm_imus arm_prefix="$(arg arm_prefix)" robot_type="$(arg robot_type)" imu_side="top"/>
     <xacro:franka_gazebo_arm_imus arm_prefix="$(arg arm_prefix)" robot_type="$(arg robot_type)" imu_side="bottom"/>

File: franka_gazebo_bringup/urdf/tmrv0_2_with_sensors.gazebo.urdf.xacro (robot description, xacro)
@@ -1,9 +1,39 @@
 <?xml version="1.0"?>
+<!--
+  Gazebo entry point for the TMR v0.2 with physical sensors.
+  Includes the franka_mobile_sensors description (base robot + sensor links),
+  ros2_control hardware interface for gazebo simulation, and Gazebo sensor plugins.
+-->
 <robot xmlns:xacro="http://www.ros.org/wiki/xacro"
        name="tmrv0_2_with_sensors_gazebo">
-  <!-- Include TMR with physical sensor links -->
-  <xacro:include filename="$(find franka_mobile_sensors)/robots/tmrv0_2_with_sensors.urdf.xacro"/>
-  <!-- Include Gazebo sensor plugin macros -->
+  <!-- ================================================================ -->
+  <!-- Macro includes                                                    -->
+  <!-- ================================================================ -->
+  <!-- TMR with physical sensor links (macro — instantiated below with gazebo=true) -->
+  <xacro:include filename="$(find franka_mobile_sensors)/robots/tmrv0_2_with_sensors.xacro"/>
+  <!-- ros2_control hardware interface -->
+  <xacro:include filename="$(find franka_hardware)/ros2_control/tmrv0_2.ros2_control.xacro"/>
+  <!-- Gazebo sensor plugin macros -->
   <xacro:include filename="$(find franka_gazebo_bringup)/urdf/sensors.xacro"/>
+  <!-- ================================================================ -->
+  <!-- Arguments                                                        -->
+  <!-- ================================================================ -->
+  <xacro:arg name="robot_type" default="tmrv0_2"/>
+  <xacro:arg name="robot_namespace" default=""/>
+  <!-- ================================================================ -->
+  <!-- Instantiate base robot + sensor suite (gazebo mode)              -->
+  <!-- ================================================================ -->
+  <xacro:tmrv0_2_with_sensors
+    robot_type="$(arg robot_type)"
+    reduced_version="false"
+    gazebo="true"
+    robot_namespace="$(arg robot_namespace)"/>
+  <!-- ================================================================ -->
+  <!-- ros2_control hardware interface (gazebo mode)                    -->
+  <!-- ================================================================ -->
+  <xacro:tmrv0_2_ros2_control
+    mobile_robot_type="$(arg robot_type)"
+    gazebo="true"
+    robot_namespace="$(arg robot_namespace)"/>
   <!-- ================= CAMERA SENSORS ================= -->
   <xacro:franka_gazebo_camera link_reference="camera_front_link"

File: franka_mobile_sensors/robots/tmrv0_2_with_sensors.urdf.xacro (robot description, xacro)
@@ -1,47 +1,25 @@
-<?xml version="1.0"?>
+<?xml version='1.0' encoding='utf-8'?>
 <robot xmlns:xacro="http://www.ros.org/wiki/xacro" name="tmrv0_2_with_sensors">
-  <!-- Include base tmrv0_2 robot -->
-  <xacro:include filename="$(find franka_description)/robots/tmrv0_2/tmrv0_2.urdf.xacro" />
-   <!-- Include RealSense D455 camera description -->
-  <xacro:include filename="$(find realsense2_description)/urdf/_d455.urdf.xacro" />
-  <!-- Include IMU description -->
-  <xacro:include filename="$(find olv_module_descriptions)/urdf/olv-imu01.urdf.xacro" />
-  <!-- Include custom SICK lidar macro (installed version has fixed "world" parent, needs wrapper for robot integration) -->
-  <xacro:include filename="$(find franka_mobile_sensors)/robots/nanoscan3/nanoscan3.xacro" />
-  <!-- Attach IMU to mounting point -->
-  <xacro:olv-imu01
-    namespace="imu"
-    parent_link="imu_mounting_point"
-    mounting_side="bottom"
-    mounting_rotation="0"/>
-  <!-- Attach cameras to mounting points -->
-  <!-- Front Camera -->
-  <xacro:sensor_d455 parent="front_mounting_point" name="camera_front"
-                     use_nominal_extrinsics="true">
-    <origin xyz="0 0 0" rpy="0 0 0"/>
-  </xacro:sensor_d455>
-  <!-- Rear Camera -->
-  <xacro:sensor_d455 parent="rear_mounting_point" name="camera_rear"
-                     use_nominal_extrinsics="true">
-    <origin xyz="0 0 0" rpy="0 0 0"/>
-  </xacro:sensor_d455>
-  <!-- Left Camera -->
-  <xacro:sensor_d455 parent="left_mounting_point" name="camera_left"
-                     use_nominal_extrinsics="true">
-    <origin xyz="0 0 0" rpy="0 0 0"/>
-  </xacro:sensor_d455>
-  <!-- Right Camera -->
-  <xacro:sensor_d455 parent="right_mounting_point" name="camera_right"
-                     use_nominal_extrinsics="true">
-    <origin xyz="0 0 0" rpy="0 0 0"/>
-  </xacro:sensor_d455>
-  <!-- Attach lidars to mounting points -->
-  <!-- Front Lidar -->
-  <xacro:lidar name="lidar_front" parent="lidar_front_mounting_point">
-    <origin xyz="0 0 0" rpy="0 0 0"/>
-  </xacro:lidar>
-  <!-- Rear Lidar -->
-  <xacro:lidar name="lidar_rear" parent="lidar_rear_mounting_point">
-    <origin xyz="0 0 0" rpy="0 0 0"/>
-  </xacro:lidar>
+  <xacro:include filename="$(find franka_mobile_sensors)/robots/tmrv0_2_with_sensors.xacro"/>
+  <!-- The ID of the robot model to be used -->
+  <xacro:arg name="robot_type" default="tmrv0_2" />
+  <!-- Should the reduced kinematic version (without caster wheels) be used? -->
+  <xacro:arg name="reduced_version" default="false" />
+  <!-- Should the robot be spawned in Gazebo? -->
+  <xacro:arg name="gazebo" default="false" />
+  <!-- The namespace of the robot -->
+  <xacro:arg name="robot_namespace" default="" />
+  <xacro:unless value="$(arg gazebo)">
+    <link name="base"/>
+    <joint name="base_joint" type="fixed">
+      <parent link="base"/>
+      <child link="base_link"/>
+      <origin rpy="0 0 0" xyz="0 0 0"/>
+    </joint>
+  </xacro:unless>
+  <xacro:tmrv0_2_with_sensors
+            robot_type="$(arg robot_type)"
+            reduced_version="$(arg reduced_version)"
+            robot_namespace="$(arg robot_namespace)"
+            gazebo="$(arg gazebo)"/>
 </robot>
