Commit message: chore: formatting

File: franka_vision_and_manipulation_kit/robots/vision_and_manipulation_kit.xacro (robot description, xacro)
@@ -94,5 +94,6 @@
     </xacro:unless>
     <!-- Attach vision kit components (wrist cameras + head camera) -->
-    <xacro:vision_kit_components left_arm_type="$(arg left_arm_type)" right_arm_type="$(arg right_arm_type)" prefix="$(arg prefix)" robotiq_use_fake_hardware="$(arg use_fake_hardware)" robotiq_include_ros2_control="$(arg ros2_control)" />
+    <xacro:vision_kit_components left_arm_type="$(arg left_arm_type)" right_arm_type="$(arg right_arm_type)"
+      prefix="$(arg prefix)" robotiq_use_fake_hardware="$(arg use_fake_hardware)" robotiq_include_ros2_control="$(arg ros2_control)" />
   </xacro:macro>
 </robot>

File: franka_vision_and_manipulation_kit/robots/vision_kit_components.xacro (robot description, xacro)
@@ -11,8 +11,13 @@
   <xacro:include filename="$(find franka_vision_and_manipulation_kit)/accessories/robotiq_gripper_with_realsense_camera.xacro" />
   <xacro:include filename="$(find zed_description)/urdf/zed_macro.urdf.xacro"/>
-  <xacro:macro name="vision_kit_components" params="left_arm_type:=fr3v2 right_arm_type:=fr3v2 prefix:='' robotiq_use_fake_hardware:=false robotiq_include_ros2_control:=true sim_gazebo:=false">
+  <xacro:macro name="vision_kit_components"
+    params="left_arm_type:=fr3v2 right_arm_type:=fr3v2 prefix:='' robotiq_use_fake_hardware:=false robotiq_include_ros2_control:=true sim_gazebo:=false">
     <!-- Robotiq Grippers with RealSense D405 wrist cameras -->
-    <xacro:robotiq_gripper_with_realsense_camera parent="left_${left_arm_type}_link8" prefix="${prefix}left_" robotiq_name="left_robotiq_gripper_hardware" robotiq_use_fake_hardware="${robotiq_use_fake_hardware}" robotiq_include_ros2_control="${robotiq_include_ros2_control}" robotiq_sim_gazebo="${sim_gazebo}" />
-    <xacro:robotiq_gripper_with_realsense_camera parent="right_${right_arm_type}_link8" prefix="${prefix}right_" robotiq_name="right_robotiq_gripper_hardware" robotiq_use_fake_hardware="${robotiq_use_fake_hardware}" robotiq_include_ros2_control="${robotiq_include_ros2_control}" robotiq_sim_gazebo="${sim_gazebo}" />
+    <xacro:robotiq_gripper_with_realsense_camera parent="left_${left_arm_type}_link8" prefix="${prefix}left_"
+      robotiq_name="left_robotiq_gripper_hardware" robotiq_use_fake_hardware="${robotiq_use_fake_hardware}"
+      robotiq_include_ros2_control="${robotiq_include_ros2_control}" robotiq_sim_gazebo="${sim_gazebo}" />
+    <xacro:robotiq_gripper_with_realsense_camera parent="right_${right_arm_type}_link8" prefix="${prefix}right_"
+      robotiq_name="right_robotiq_gripper_hardware" robotiq_use_fake_hardware="${robotiq_use_fake_hardware}"
+      robotiq_include_ros2_control="${robotiq_include_ros2_control}" robotiq_sim_gazebo="${sim_gazebo}" />
     <!-- ZED Mini head camera -->
     <xacro:zed_camera name="${prefix}head" model="zedm" custom_baseline="0.0" enable_gnss="false">
