Commit message: refactor: put cartesian_velocity_interface_prefix into controller.yaml files only, remove use_fake_hardware option

File: franka_mobile_fr3_duo_moveit_config/urdf/mobile_fr3_duo_v0_2.moveit.urdf.xacro (robot description, xacro)
@@ -53,5 +53,5 @@
         <axis xyz="1 0 0" />
         <origin rpy="0 0 0" xyz="0 0 0" />
-        <limit lower="-1" upper="1" effort="1000" velocity="2" />
+        <limit lower="-10" upper="10" effort="1000" velocity="2" />
     </joint>
     <link name="virtual_x">
@@ -86,5 +86,5 @@
         <axis xyz="0 1 0" />
         <origin rpy="0 0 0" xyz="0 0 0" />
-        <limit lower="-1" upper="1" effort="1000" velocity="2" />
+        <limit lower="-10" upper="10" effort="1000" velocity="2" />
     </joint>
     <joint name="planar_theta" type="revolute">
