Commit message: joint_state_broadcaster and fr3_zrm_controller is active
gravity compensation_example_controller is inactive

File: fr3_delivery_sim/urdf/fr3_vision_env.urdf.xacro (robot description, xacro)
@@ -1,44 +1,42 @@
 <?xml version="1.0"?>
 <!--
-  fr3_vision_env.urdf.xacro  — Phase 4 "Gazebo Physics" (world-link-collision fix)
-  ROOT CAUSE of previous crash:
-    When gazebo:=true, franka_description's franka_robot.xacro already emits:
-        <link name="world"/>
-        <joint name="world_joint" type="fixed">
-          <parent link="world"/> <child link="base"/>
-        </joint>
-    Our file was also declaring <link name="world"/>, making it non-unique.
-    URDF is strict: duplicate link names are a fatal parse error.
-  FIX:
-    Remove our <link name="world"/> and <joint name="robot_to_world"> entirely.
-    The upstream xacro provides the world anchor when gazebo:=true.
-    The camera is attached to fr3_link0 (unchanged).
+  fr3_vision_env.urdf.xacro  —  Phase 4 FINAL
+  =============================================
+  Adds the overhead RGBD camera to the standard FR3 description.
+  IMPORTANT — world link:
+    When gazebo:=true (which we always pass from sim.launch.py), the included
+    franka_description xacro ALREADY generates:
+      <link name="world"/>
+      <joint name="world_joint" type="fixed"> world → base </joint>
+    Do NOT redeclare world here — that causes a fatal "link is not unique" error.
+    The camera joint is parented to fr3_link0, which is already in the tree.
+  Args passed from sim.launch.py:
+    hand:=true
+    ros2_control:=true
+    gazebo:=true        ← triggers world link + Gazebo plugin in franka_description
+    use_fake_hardware:=false
+    fake_sensor_commands:=false
 -->
 <robot xmlns:xacro="http://www.ros.org/wiki/xacro" name="fr3_vision">
-  <!-- ── Parameters forwarded to franka_description ──────────────────────── -->
+  <!-- ── Declare all args so xacro doesn't warn about undeclared overrides ── -->
   <xacro:arg name="hand"                 default="true"/>
   <xacro:arg name="ros2_control"         default="true"/>
+  <xacro:arg name="gazebo"               default="true"/>
   <xacro:arg name="use_fake_hardware"    default="false"/>
   <xacro:arg name="fake_sensor_commands" default="false"/>
-  <xacro:arg name="gazebo"               default="true"/>
-  <xacro:arg name="gazebo_effort"        default="false"/>
-  <!--
-    This include, with gazebo:=true, injects:
-      • All FR3 links/joints/meshes/inertials
-      • <link name="world"/> + world→base fixed joint  ← DO NOT duplicate
-      • <ros2_control> block using ign_ros2_control/IgnitionSystem
-      • <gazebo> plugin tag for IgnitionROS2ControlPlugin
+  <xacro:arg name="robot_ip"             default="dont-care"/>
+  <xacro:arg name="robot_type"           default="fr3"/>
+  <!-- ── Official FR3 arm description ──────────────────────────────────────
+       All args are forwarded through to fr3.urdf.xacro via the command-line
+       xacro argument mechanism (xacro shares args across includes).
+       With gazebo:=true this also generates:
+         - <ros2_control> hardware block  (gz_ros2_control/GazeboSimSystem)
+         - <gazebo><plugin>               (ign_ros2_control/IgnitionROS2ControlPlugin)
+         - <link name="world"/>  +  world_joint
   -->
   <xacro:include filename="$(find franka_description)/robots/fr3/fr3.urdf.xacro"/>
-  <!--
-    ╔══════════════════════════════════════════════════════════════╗
-    ║  NO <link name="world"/> here — franka_description owns it  ║
-    ╚══════════════════════════════════════════════════════════════╝
-    Camera is parented to fr3_link0 (the robot's base footprint link)
-    which is already connected to world via the upstream xacro.
-  -->
   <!-- ── Overhead camera link ───────────────────────────────────────────────
-    Must have <inertial> — Ignition collapses mass-less links into their
-    parent during URDF→SDF conversion, silently deleting any sensor on them.
+       MUST have <inertial> — Ignition Gazebo collapses massless links into
+       their parent during URDF→SDF conversion, silently deleting the sensor.
   -->
   <link name="camera_link">
@@ -58,5 +56,8 @@
     </collision>
   </link>
-  <!-- 0.5 m forward, 1.0 m up from robot base, pitched 90° to look straight down -->
+  <!--
+    Mount the camera 0.5 m forward and 1.0 m above fr3_link0,
+    pitched 90° so it looks straight down.
+  -->
   <joint name="camera_joint" type="fixed">
     <parent link="fr3_link0"/>
@@ -64,13 +65,10 @@
     <origin xyz="0.5 0.0 1.0" rpy="0 ${pi/2} 0"/>
   </joint>
-  <!-- ── Ignition Gazebo RGBD camera sensor ────────────────────────────────
-    Bridged topics (via ros_gz_bridge in launch file):
-      /camera/image          RGB frames
-      /camera/depth_image    float32 depth in metres
-      /camera/camera_info    intrinsic matrix K
-      /camera/points         PointCloud2
+  <!-- ── Ignition Gazebo RGBD sensor ───────────────────────────────────────
+       Publishes on /camera/{image,depth_image,points,camera_info}.
+       Bridged to ROS 2 topics by ros_gz_bridge in sim.launch.py.
   -->
   <gazebo reference="camera_link">
-    <sensor type="rgbd_camera" name="overhead_rgbd">
+    <sensor type="rgbd_camera" name="realsense_d435">
       <ignition_frame_id>camera_link</ignition_frame_id>
       <always_on>1</always_on>
@@ -78,5 +76,5 @@
       <visualize>1</visualize>
       <topic>/camera</topic>
-      <camera name="overhead_rgbd_cam">
+      <camera name="overhead_rgbd">
         <horizontal_fov>1.2</horizontal_fov>
         <image>

Commit message: added pick.py for troubleshooting

File: fr3_delivery_sim/urdf/fr3_vision_env.urdf.xacro (robot description, xacro)
@@ -94,3 +94,39 @@
     </sensor>
   </gazebo>
+  <!-- ── Gripper finger control (bypasses gz_ros2_control mimic bug #343) ──────
+       fr3_finger_joint1 is the mimic LEADER; fr3_finger_joint2 mimics it in the
+       URDF, which makes gz_ros2_control refuse to actuate joint1 via its position
+       command interface (https://github.com/ros-controls/gz_ros2_control/issues/343).
+       Ignition also does not enforce URDF <mimic> on its own, so joint2 follows
+       nothing. We therefore drive BOTH fingers directly with Ignition's native
+       JointPositionController and command them to the same value from pick.py.
+       NOTE: the fr3_gripper ros2_control controller must NOT be spawned, or it
+       will fight these plugins for fr3_finger_joint1. (Removed in sim_launch.py.)
+  -->
+  <gazebo>
+    <plugin filename="ignition-gazebo-joint-position-controller-system"
+            name="ignition::gazebo::systems::JointPositionController">
+      <joint_name>fr3_finger_joint1</joint_name>
+      <topic>/fr3_finger_joint1_cmd</topic>
+      <p_gain>2000</p_gain>
+      <i_gain>15</i_gain>
+      <d_gain>40</d_gain>
+      <i_max>100</i_max>
+      <i_min>-100</i_min>
+      <cmd_max>100</cmd_max>
+      <cmd_min>-100</cmd_min>
+    </plugin>
+    <plugin filename="ignition-gazebo-joint-position-controller-system"
+            name="ignition::gazebo::systems::JointPositionController">
+      <joint_name>fr3_finger_joint2</joint_name>
+      <topic>/fr3_finger_joint2_cmd</topic>
+      <p_gain>2000</p_gain>
+      <i_gain>15</i_gain>
+      <d_gain>40</d_gain>
+      <i_max>100</i_max>
+      <i_min>-100</i_min>
+      <cmd_max>100</cmd_max>
+      <cmd_min>-100</cmd_min>
+    </plugin>
+  </gazebo>
 </robot>
