Commit message: test: Adding tests for gravity compensation model refactor: Move gravity compensation system to franka_gazebo_hardware package

File: franka_hardware/ros2_control/fr3_duo.ros2_control.xacro (robot description, xacro)
@@ -29,5 +29,10 @@
         </xacro:if>
         <xacro:if value="${gazebo}">
-          <plugin>gz_ros2_control/GazeboSimSystem</plugin>
+          <xacro:if value="${gazebo_effort}">
+            <plugin>franka_gazebo_hardware/GazeboGravityCompensationSystem</plugin>
+          </xacro:if>
+          <xacro:unless value="${gazebo_effort}">
+            <plugin>gz_ros2_control/GazeboSimSystem</plugin>
+          </xacro:unless>
         </xacro:if>
         <xacro:if value="${use_fake_hardware == 0 and gazebo == 0}">

File: franka_hardware/ros2_control/franka_ros2_control_macros.xacro (robot description, xacro)
@@ -104,6 +104,20 @@
   <xacro:macro name="configure_passive_mobile_base_joints" params="include_spine:=0">
     <xacro:if value="${include_spine}">
-      <!-- Spine -->
-      <xacro:passive_joint joint_name="franka_spine_vertical_joint"/>
+      <!-- Spine: the prismatic spine carries the full upper-body weight. With
+           gravity enabled globally in Gazebo it would collapse unless actively
+           held, so (this macro is only instantiated under Gazebo) it gets a
+           position command interface and is held at its initial height by
+           spine_joint_trajectory_controller. gz_ros2_control issue #343
+           (position+velocity command interface bug) does not apply here: the
+           spine declares only a single position command interface. -->
+      <joint name="franka_spine_vertical_joint">
+        <command_interface name="position"/>
+        <state_interface name="position">
+          <param name="initial_value">0.0</param>
+        </state_interface>
+        <state_interface name="velocity">
+          <param name="initial_value">0.0</param>
+        </state_interface>
+      </joint>
     </xacro:if>
     <!-- Rocker Arm -->

File: franka_hardware/ros2_control/mobile_fr3_duo.ros2_control.xacro (robot description, xacro)
@@ -32,5 +32,10 @@
         </xacro:if>
         <xacro:if value="${gazebo}">
-          <plugin>gz_ros2_control/GazeboSimSystem</plugin>
+          <xacro:if value="${gazebo_effort}">
+            <plugin>franka_gazebo_hardware/GazeboGravityCompensationSystem</plugin>
+          </xacro:if>
+          <xacro:unless value="${gazebo_effort}">
+            <plugin>gz_ros2_control/GazeboSimSystem</plugin>
+          </xacro:unless>
         </xacro:if>
         <xacro:if value="${use_fake_hardware == 0 and gazebo == 0}">
