Commit message: fix: make robot_ip and use_rviz launch arguments of tmrv0_2 and publish sensor TF without RViz
tmrv0_2.launch.py read robot_ip and use_rviz only from the config file, so
they could not be set on the command line. Both are now launch arguments that
override the config file when given.

franka_mobile_sensors started the robot_state_publisher for the sensor frames
only together with RViz, so start_rviz:=false dropped the lidar and camera
frames from TF. With RViz off, franka_mobile_sensors.launch.py now starts a
robot_state_publisher in the sensors namespace (publish_sensor_tf, default
true). The namespace keeps its URDF off /robot_description and the node off
/joint_states, so it can run next to tmrv0_2.launch.py.

The sensor entry points no longer add the fixed base -> base_link joint, which
competed with the swerve odometry; the trees start at base_link like the
bringup description and the Gazebo wrapper.

franka_bringup gains a test that every joint of tmrv0_2.urdf.xacro exists in
tmrv0_2_with_sensors.urdf.xacro with the same type, parent, child and origin,
since both publish the base frames side by side. franka_mobile_sensors declares
joint_state_publisher_gui, robot_state_publisher, launch and launch_ros.

File: franka_description_extensions/franka_mobile_sensors/robots/mobile_fr3_duo_v0_2_with_sensors.urdf.xacro (robot description, xacro)
@@ -36,10 +36,4 @@
   <!-- Should the arms be used? -->
   <xacro:arg name="use_arms" default="true" />
-  <link name="base"/>
-  <joint name="base_joint" type="fixed">
-    <parent link="base"/>
-    <child link="base_link"/>
-    <origin rpy="0 0 0" xyz="0 0 0"/>
-  </joint>
   <xacro:mobile_fr3_duo_v0_2_with_sensors
         robot_types="$(arg robot_types)"

File: franka_description_extensions/franka_mobile_sensors/robots/tmrv0_2_with_sensors.urdf.xacro (robot description, xacro)
@@ -8,10 +8,4 @@
   <!-- The namespace of the robot -->
   <xacro:arg name="robot_namespace" default="" />
-  <link name="base"/>
-  <joint name="base_joint" type="fixed">
-    <parent link="base"/>
-    <child link="base_link"/>
-    <origin rpy="0 0 0" xyz="0 0 0"/>
-  </joint>
   <xacro:tmrv0_2_with_sensors
             robot_type="$(arg robot_type)"
